Commit message: Migrated to dashing
Signed-off-by: Gonzalo de Pedro <gonzalo@depedro.com.ar>

File: velodyne_description/urdf/example.urdf (robot description, URDF)
Before this commit: robot example, 4 links, 3 joints
Links:
- added link velodyne2, mass 0.01; visual mesh filename=package://velodyne_description/meshes/HDL32E_scan.dae
- added link velodyne2_base_link, mass 1.0; collision cylinder length=0.14424 radius=0.04267; visual mesh filename=package://velodyne_description/meshes/HDL32E_base.dae
Joints:
- added joint velodyne2_base_mount_joint: type fixed, parent base_link, child velodyne2_base_link, origin xyz=0 0 0.6 rpy=0 0 0
- added joint velodyne2_base_scan_joint: type fixed, parent velodyne2_base_link, child velodyne2, origin xyz=0 0 0.09081 rpy=0 0 0
