Commit message: Misc updates.
Signed-off-by: Michel Hidalgo <michel@ekumenlabs.com>

File: velodyne_description/urdf/VLP-32C.urdf.xacro (robot description, xacro)
@@ -2,5 +2,5 @@
 <robot xmlns:xacro="http://www.ros.org/wiki/xacro" name="VLP-32C">
   <xacro:property name="M_PI" value="3.1415926535897931"/>
-  <xacro:macro name="VLP-32C" params="*origin parent:=base_link name:=velodyne topic:=/velodyne_points hz:=10 lasers:=32 samples:=1200 collision_range:=0.3 min_range:=0.9 max_range:=200.0 noise:=0.008 min_angle:=-${M_PI} max_angle:=${M_PI} gpu:=false">
+  <xacro:macro name="VLP-32C" params="*origin parent:=base_link name:=velodyne topic:=/velodyne_points hz:=10 lasers:=32 samples:=1200 collision_range:=0.3 min_range:=0.4 max_range:=200.0 noise:=0.008 min_angle:=-${M_PI} max_angle:=${M_PI} gpu:=false">
     <joint name="${name}_base_mount_joint" type="fixed">
       <xacro:insert_block name="origin"/>
@@ -89,12 +89,12 @@
               <vertical>
                 <angles>
-                  ${-25.000*M_PI/180.0}  ${-15.639*M_PI/180.0}  ${-11.310*M_PI/180.0}  ${-8.843*M_PI/180.0}
-                  ${-7.254*M_PI/180.0}   ${-6.148*M_PI/180.0}   ${-5.333*M_PI/180.0}   ${-4.667*M_PI/180.0}
-                  ${-4.000*M_PI/180.0}   ${-3.667 *M_PI/180.0}  ${-3.333 *M_PI/180.0}  ${-3.000 *M_PI/180.0}
-                  ${-2.667 *M_PI/180.0}  ${-2.333 *M_PI/180.0}  ${-2.000 *M_PI/180.0}  ${-1.667*M_PI/180.0}
-                  ${-1.333*M_PI/180.0}   ${-1.000 *M_PI/180.0}  ${-0.667 *M_PI/180.0}  ${-0.333 *M_PI/180.0}
-                  ${0.000 *M_PI/180.0}   ${0.333 *M_PI/180.0}   ${ 0.667 *M_PI/180.0}  ${1.000*M_PI/180.0}
-                  ${1.333*M_PI/180.0}    ${1.667*M_PI/180.0}    ${2.333*M_PI/180.0}    ${3.333*M_PI/180.0}
-                  ${4.667*M_PI/180.0}    ${7.000*M_PI/180.0}    ${10.333*M_PI/180.0}   ${15.000*M_PI/180.0}
+                  ${-25.000 * M_PI / 180.0}  ${-15.639 * M_PI / 180.0}  ${-11.310 * M_PI / 180.0}  ${-8.843 * M_PI / 180.0}
+                  ${ -7.254 * M_PI / 180.0}  ${ -6.148 * M_PI / 180.0}  ${ -5.333 * M_PI / 180.0}  ${-4.667 * M_PI / 180.0}
+                  ${ -4.000 * M_PI / 180.0}  ${ -3.667 * M_PI / 180.0}  ${ -3.333 * M_PI / 180.0}  ${-3.000 * M_PI / 180.0}
+                  ${ -2.667 * M_PI / 180.0}  ${ -2.333 * M_PI / 180.0}  ${ -2.000 * M_PI / 180.0}  ${-1.667 * M_PI / 180.0}
+                  ${ -1.333 * M_PI / 180.0}  ${ -1.000 * M_PI / 180.0}  ${ -0.667 * M_PI / 180.0}  ${-0.333 * M_PI / 180.0}
+                  ${  0.000 * M_PI / 180.0}  ${  0.333 * M_PI / 180.0}  ${  0.667 * M_PI / 180.0}  ${ 1.000 * M_PI / 180.0}
+                  ${  1.333 * M_PI / 180.0}  ${  1.667 * M_PI / 180.0}  ${  2.333 * M_PI / 180.0}  ${ 3.333 * M_PI / 180.0}
+                  ${  4.667 * M_PI / 180.0}  ${  7.000 * M_PI / 180.0}  ${ 10.333 * M_PI / 180.0}  ${15.000 * M_PI / 180.0}
                 </angles>
               </vertical>
@@ -143,12 +143,12 @@
               <vertical>
                 <angles>
-                  ${-25.000*M_PI/180.0}  ${-15.639*M_PI/180.0}  ${-11.310*M_PI/180.0}  ${-8.843*M_PI/180.0}
-                  ${-7.254*M_PI/180.0}   ${-6.148*M_PI/180.0}   ${-5.333*M_PI/180.0}   ${-4.667*M_PI/180.0}
-                  ${-4.000*M_PI/180.0}   ${-3.667 *M_PI/180.0}  ${-3.333 *M_PI/180.0}  ${-3.000 *M_PI/180.0}
-                  ${-2.667 *M_PI/180.0}  ${-2.333 *M_PI/180.0}  ${-2.000 *M_PI/180.0}  ${-1.667*M_PI/180.0}
-                  ${-1.333*M_PI/180.0}   ${-1.000 *M_PI/180.0}  ${-0.667 *M_PI/180.0}  ${-0.333 *M_PI/180.0}
-                  ${0.000 *M_PI/180.0}   ${0.333 *M_PI/180.0}   ${ 0.667 *M_PI/180.0}  ${1.000*M_PI/180.0}
-                  ${1.333*M_PI/180.0}    ${1.667*M_PI/180.0}    ${2.333*M_PI/180.0}    ${3.333*M_PI/180.0}
-                  ${4.667*M_PI/180.0}    ${7.000*M_PI/180.0}    ${10.333*M_PI/180.0}   ${15.000*M_PI/180.0}
+                  ${-25.000 * M_PI / 180.0}  ${-15.639 * M_PI / 180.0}  ${-11.310 * M_PI / 180.0}  ${-8.843 * M_PI / 180.0}
+                  ${ -7.254 * M_PI / 180.0}  ${ -6.148 * M_PI / 180.0}  ${ -5.333 * M_PI / 180.0}  ${-4.667 * M_PI / 180.0}
+                  ${ -4.000 * M_PI / 180.0}  ${ -3.667 * M_PI / 180.0}  ${ -3.333 * M_PI / 180.0}  ${-3.000 * M_PI / 180.0}
+                  ${ -2.667 * M_PI / 180.0}  ${ -2.333 * M_PI / 180.0}  ${ -2.000 * M_PI / 180.0}  ${-1.667 * M_PI / 180.0}
+                  ${ -1.333 * M_PI / 180.0}  ${ -1.000 * M_PI / 180.0}  ${ -0.667 * M_PI / 180.0}  ${-0.333 * M_PI / 180.0}
+                  ${  0.000 * M_PI / 180.0}  ${  0.333 * M_PI / 180.0}  ${  0.667 * M_PI / 180.0}  ${ 1.000 * M_PI / 180.0}
+                  ${  1.333 * M_PI / 180.0}  ${  1.667 * M_PI / 180.0}  ${  2.333 * M_PI / 180.0}  ${ 3.333 * M_PI / 180.0}
+                  ${  4.667 * M_PI / 180.0}  ${  7.000 * M_PI / 180.0}  ${ 10.333 * M_PI / 180.0}  ${15.000 * M_PI / 180.0}
                 </angles>
               </vertical>
