Commit message: Add support for the VLP-32C Ultra Puck model.
Signed-off-by: Michel Hidalgo <michel@ekumenlabs.com>

File: velodyne_description/urdf/example.urdf.xacro (robot description, xacro)
@@ -34,7 +34,11 @@
     <origin xyz="0 0 0.4" rpy="0 0 0" />
   </VLP-16>
-  <xacro:include filename="$(find velodyne_description)/urdf/HDL-32E.urdf.xacro"/>
-  <HDL-32E parent="base_link" name="velodyne2" topic="/velodyne_points2" hz="10" samples="220" gpu="${gpu}">
+  <xacro:include filename="$(find velodyne_description)/urdf/HDL-32E.urdf.xacro"/> -->
+   <HDL-32E parent="base_link" name="velodyne2" topic="/velodyne_points2" hz="10" samples="220" gpu="${gpu}">
     <origin xyz="0 0 0.6" rpy="0 0 0" />
   </HDL-32E>
+  <xacro:include filename="$(find velodyne_description)/urdf/VLP-32C.urdf.xacro"/>
+  <VLP-32C parent="base_link" name="velodyne3" topic="/velodyne_points3" hz="10" samples="1200" gpu="${gpu}">
+  <origin xyz="0 0 0.8" rpy="0 0 0" />
+  </VLP-32C>
 </robot>

Commit message: Clean up velodyne_description example.urdf.xacro
Signed-off-by: Michel Hidalgo <michel@ekumenlabs.com>

File: velodyne_description/urdf/example.urdf.xacro (robot description, xacro)
@@ -34,5 +34,5 @@
     <origin xyz="0 0 0.4" rpy="0 0 0" />
   </VLP-16>
-  <xacro:include filename="$(find velodyne_description)/urdf/HDL-32E.urdf.xacro"/> -->
+  <xacro:include filename="$(find velodyne_description)/urdf/HDL-32E.urdf.xacro"/>
    <HDL-32E parent="base_link" name="velodyne2" topic="/velodyne_points2" hz="10" samples="220" gpu="${gpu}">
     <origin xyz="0 0 0.6" rpy="0 0 0" />
@@ -40,5 +40,5 @@
   <xacro:include filename="$(find velodyne_description)/urdf/VLP-32C.urdf.xacro"/>
   <VLP-32C parent="base_link" name="velodyne3" topic="/velodyne_points3" hz="10" samples="1200" gpu="${gpu}">
-  <origin xyz="0 0 0.8" rpy="0 0 0" />
+    <origin xyz="0 0 0.8" rpy="0 0 0" />
   </VLP-32C>
 </robot>

Commit message: Add support for the VLP-32C Ultra Puck model. (#1)
Signed-off-by: Michel Hidalgo <michel@ekumenlabs.com>

File: velodyne_description/urdf/example.urdf.xacro (robot description, xacro)
@@ -35,6 +35,10 @@
   </VLP-16>
   <xacro:include filename="$(find velodyne_description)/urdf/HDL-32E.urdf.xacro"/>
-  <HDL-32E parent="base_link" name="velodyne2" topic="/velodyne_points2" hz="10" samples="220" gpu="${gpu}">
+   <HDL-32E parent="base_link" name="velodyne2" topic="/velodyne_points2" hz="10" samples="220" gpu="${gpu}">
     <origin xyz="0 0 0.6" rpy="0 0 0" />
   </HDL-32E>
+  <xacro:include filename="$(find velodyne_description)/urdf/VLP-32C.urdf.xacro"/>
+  <VLP-32C parent="base_link" name="velodyne3" topic="/velodyne_points3" hz="10" samples="1200" gpu="${gpu}">
+    <origin xyz="0 0 0.8" rpy="0 0 0" />
+  </VLP-32C>
 </robot>
